File: Arduino_LedStrip.sch (KiCad schematic (older format))
At the start: 26 parts, among them J1 Conn_L, J2 Conn_R, J3 LED0, J4 LED1, J5 LED_WS2812B, J6 Barrel_Jack, Q1 IRFZ44N, Q2 IRFZ44N, Q3 IRFZ44N, Q4 IRFZ44N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

Commit message: Routing PCB
Parts:
- added J10, J7, J8, J9: Screw_Terminal_01x01, Mounting_Holes:MountingHole_3.2mm_M3, symbol Screw_Terminal_01x01
Connections:
- net +5V: now also J5.3 (Pin_3); no longer J5.1 (Pin_1)
- net GND: now also J5.1 (Pin_1); no longer J5.3 (Pin_3)
- net ar_LED0_G: now also A1.12 (D9), J2.4 (Pin_4); no longer A1.13 (D10), J2.3 (Pin_3)
- net ar_LED0_R: now also A1.13 (D10), J2.3 (Pin_3); no longer A1.12 (D9), J2.4 (Pin_4)
- no-connect marks 0 -> 4
Other:
- moved on the sheet: C1
Changed lines of the file:
@@
 Text Label 2350 1950 0    60   ~ 0
 ar_Aref
+Text Label 1350 2550 2    60   ~ 0
+ar_LED0_R
 Text Label 1350 2450 2    60   ~ 0
-ar_LED0_R
-Text Label 1350 2550 2    60   ~ 0
 ar_LED0_G
 Text Label 1350 2650 2    60   ~ 0
@@
 Text Label 7350 3300 2    60   ~ 0
 ar_Din_LEDWS
+Text Label 7350 2700 2    60   ~ 0
+ar_LED0_R
 Text Label 7350 2800 2    60   ~ 0
-ar_LED0_R
-Text Label 7350 2700 2    60   ~ 0
 ar_LED0_G
 Text Label 7350 2600 2    60   ~ 0
@@
 F 3 "" H 4100 3700 50  0001 C CNN
 	1    4100 3700
-	-1   0    0    -1
+	-1   0    0    1
 $EndComp
 Text Label 3900 3700 2    60   ~ 0
@@
 L CP C1
 U 1 1 5A116536
-P 1050 3700
-F 0 "C1" H 1075 3800 50  0000 L CNN
-F 1 "10u" H 1075 3600 50  0000 L CNN
-F 2 "Capacitors_ThroughHole:CP_Radial_D8.0mm_P3.50mm" H 1088 3550 50  0001 C CNN
-F 3 "" H 1050 3700 50  0001 C CNN
-	1    1050 3700
+P 750 3700
+F 0 "C1" H 775 3800 50  0000 L CNN
+F 1 "10u" H 775 3600 50  0000 L CNN
+F 2 "Capacitors_ThroughHole:CP_Radial_D8.0mm_P3.50mm" H 788 3550 50  0001 C CNN
+F 3 "" H 750 3700 50  0001 C CNN
+	1    750  3700
 	1    0    0    -1
 $EndComp
@@
 L +12V #PWR028
 U 1 1 5A1165A3
-P 1050 3550
-F 0 "#PWR028" H 1050 3400 50  0001 C CNN
-F 1 "+12V" H 1050 3690 50  0000 C CNN
-F 2 "" H 1050 3550 50  0001 C CNN
-F 3 "" H 1050 3550 50  0001 C CNN
-	1    1050 3550
+P 750 3550
+F 0 "#PWR028" H 750 3400 50  0001 C CNN
+F 1 "+12V" H 750 3690 50  0000 C CNN
+F 2 "" H 750 3550 50  0001 C CNN
+F 3 "" H 750 3550 50  0001 C CNN
+	1    750  3550
 	1    0    0    -1
 $EndComp
@@
 L GND #PWR029
 U 1 1 5A1165FC
-P 1050 3850
-F 0 "#PWR029" H 1050 3600 50  0001 C CNN
-F 1 "GND" H 1050 3700 50  0000 C CNN
-F 2 "" H 1050 3850 50  0001 C CNN
-F 3 "" H 1050 3850 50  0001 C CNN
-	1    1050 3850
+P 750 3850
+F 0 "#PWR029" H 750 3600 50  0001 C CNN
+F 1 "GND" H 750 3700 50  0000 C CNN
+F 2 "" H 750 3850 50  0001 C CNN
+F 3 "" H 750 3850 50  0001 C CNN
+	1    750  3850
 	1    0    0    -1
 $EndComp
@@
 	-1   0    0    1
 $EndComp
+$Comp
+L Screw_Terminal_01x01 J9
+U 1 1 5A11E95E
+P 1800 3900
+F 0 "J9" H 1800 4000 50  0000 C CNN
+F 1 "Screw_Terminal_01x01" H 1800 3800 50  0000 C CNN
+F 2 "Mounting_Holes:MountingHole_3.2mm_M3" H 1800 3900 50  0001 C CNN
+F 3 "" H 1800 3900 50  0001 C CNN
+	1    1800 3900
+	1    0    0    -1
+$EndComp
+$Comp
+L Screw_Terminal_01x01 J7
+U 1 1 5A11EA74
+P 1800 3650
+F 0 "J7" H 1800 3750 50  0000 C CNN
+F 1 "Screw_Terminal_01x01" H 1800 3550 50  0000 C CNN
+F 2 "Mounting_Holes:MountingHole_3.2mm_M3" H 1800 3650 50  0001 C CNN
+F 3 "" H 1800 3650 50  0001 C CNN
+	1    1800 3650
+	1    0    0    -1
+$EndComp
+$Comp
+L Screw_Terminal_01x01 J8
+U 1 1 5A11EE66
+P 2650 3650
+F 0 "J8" H 2650 3750 50  0000 C CNN
+F 1 "Screw_Terminal_01x01" H 2650 3550 50  0000 C CNN
+F 2 "Mounting_Holes:MountingHole_3.2mm_M3" H 2650 3650 50  0001 C CNN
+F 3 "" H 2650 3650 50  0001 C CNN
+	1    2650 3650
+	1    0    0    -1
+$EndComp
+$Comp
+L Screw_Terminal_01x01 J10
+U 1 1 5A11EEF9
+P 2650 3900
+F 0 "J10" H 2650 4000 50  0000 C CNN
+F 1 "Screw_Terminal_01x01" H 2650 3800 50  0000 C CNN
+F 2 "Mounting_Holes:MountingHole_3.2mm_M3" H 2650 3900 50  0001 C CNN
+F 3 "" H 2650 3900 50  0001 C CNN
+	1    2650 3900
+	1    0    0    -1
+$EndComp
+NoConn ~ 1600 3650
+NoConn ~ 2450 3650
+NoConn ~ 2450 3900
+NoConn ~ 1600 3900
 $EndSCHEMATC
