File: KiCad/Arduino_LedStrip.kicad_pcb (KiCad board)
At the start: 2 copper layers, 48 x 60.5 mm, 35 parts, among them J1 Conn_L, J10 Screw_Terminal_01x01, J2 Conn_R, J3 LED0, J4 LED1, J5 LED_WS2812B, J6 Barrel_Jack, J7 Screw_Terminal_01x01, J8 Screw_Terminal_01x01, J9 Screw_Terminal_01x01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

Commit message: Update folder paths. Add Wemos.
Parts:
- removed J1: Conn_L, Pin_Headers:Pin_Header_Straight_1x15_Pitch2.54mm
- removed J10: Screw_Terminal_01x01, Mounting_Holes:MountingHole_3.2mm_M3
- removed J2: Conn_R, Pin_Headers:Pin_Header_Straight_1x15_Pitch2.54mm
- added R12: *1kor0, Resistors_SMD:R_0603_HandSoldering, F.Cu at (133.8, 100.2)
- added R9: *1kor0, Resistors_SMD:R_0603_HandSoldering, F.Cu at (133.8, 91.8)
- added U2: L7805, TO_SOT_Packages_THT:TO-220-3_Vertical, F.Cu at (153.5, 91.2)
- added U3: WeMos_mini, GoInK13:D1_mini_board, F.Cu at (151.1, 69.1)
- moved R7 1.50 mm to (136.2, 90.5)
- moved R11 0.25 mm to (128.5, 97.2)
Connections:
- A1 pad 17: /3V3 -> +3V3
- A1 pad 18: /ar_Aref -> +3V3
- A1 pad 30: /Vin -> +12V
- C1 pad 1: +12V -> VCC
- J3 pad 1: +12V -> VCC
- J4 pad 1: +12V -> VCC
- J5 pad 3: +12V -> VCC
- J6 pad 1: +12V -> VCC
- R10 pad 1: /Vin -> +12V
- R10 pad 2: +12V -> VCC
- R11 pad 1: +12V -> VCC
- RV1 pad 3: +5V -> +3V3
- SW1 pad 2: /ar_A1_D15 -> Net-(R9-Pad2)
- SW2 pad 2: /ar_A2_D16 -> Net-(R12-Pad2)
Routing:
- net VCC: track 0.00 -> 113.5 mm, vias 0 -> 1
- net /Vin: track 57.6 -> 0.00 mm, vias 1 -> 0
- net +5V: track 54.8 -> 106.9 mm, vias 0 -> 4
- net +12V: track 113.8 -> 64.1 mm, vias 1 -> 2
- net +3V3: track 0.00 -> 35.3 mm, vias 0 -> 1
- net /ar_LED0_R: track 45.1 -> 67.3 mm, vias 0 -> 4
- net /ar_LED0_G: track 52.1 -> 68.0 mm, vias 0 -> 4
- net GND: track 328.9 -> 341.0 mm, vias 30 -> 33
- net /ar_IR: track 96.5 -> 104.5 mm, vias 0 -> 1
- net /ar_LED1_B: track 45.0 -> 50.2 mm
- net /ar_Reset1: track 4.00 -> 0.00 mm
- net /ar_LED_BuiltIn: track 4.00 -> 0.00 mm
- net /ar_Aref: track 4.00 -> 0.00 mm
- net /ar_A7: track 4.00 -> 0.00 mm
- net /ar_A6: track 4.00 -> 0.00 mm
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- added copper zone on F.Cu, net VCC
Other:
- board text added: "* 1kor0 : Connect 1kΩ if Wemos (3V3) Connect 0Ω if arduino (5V) LED_WS2812B needs 5V as input, else 12V"
- board text added: "+"
- board text added: "-"
- board text removed: "LED_BuiltIn"
