File: KiCad/Arduino_LedStrip.kicad_pcb (KiCad board)
At the start: 2 copper layers, 48 x 60.5 mm, 36 parts, among them J3 LED0, J4 LED1, J5 LED_WS2812B, J6 Barrel_Jack, J7 Screw_Terminal_01x01, J8 Screw_Terminal_01x01, J9 Screw_Terminal_01x01, Q1 IRFZ44N, Q2 IRFZ44N, Q3 IRFZ44N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

Commit message: Up 3D : Add Arduino Nano.
Parts:
- A1: footprint Modules:Arduino_Nano -> Module:Arduino_Nano
Changed lines of the file:
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@@
     (add_net VCC)
   )
-  (module TO_SOT_Packages_THT:TO-220-3_Vertical (layer F.Cu)
-    (at 161 101 270)
-    (descr "TO-220-3, Vertical, RM 2.54mm")
-    (tags "TO-220-3 Vertical RM 2.54mm")
-    (fp_text reference Q4 (at 2.54 -3.62 270) (layer F.SilkS)
-      (effects (font (size 1 1) (thickness 0.15)))
-    )
-    (fp_text value IRFZ44N (at 2.54 3.92 270) (layer F.Fab) hide
-      (effects (font (size 1 1) (thickness 0.15)))
-    )
-    (fp_text user %R (at 2.54 -3.62 270) (layer F.Fab) hide
-      (effects (font (size 1 1) (thickness 0.15)))
-    )
-    (fp_line (start -2.46 -2.5) (end -2.46 1.9) (layer F.Fab) (width 0.1))
-    (fp_line (start -2.46 1.9) (end 7.54 1.9) (layer F.Fab) (width 0.1))
-    (fp_line (start 7.54 1.9) (end 7.54 -2.5) (layer F.Fab) (width 0.1))
-    (fp_line (start 7.54 -2.5) (end -2.46 -2.5) (layer F.Fab) (width 0.1))
-    (fp_line (start -2.46 -1.23) (end 7.54 -1.23) (layer F.Fab) (width 0.1))
-    (fp_line (start 0.69 -2.5) (end 0.69 -1.23) (layer F.Fab) (width 0.1))
-    (fp_line (start 4.39 -2.5) (end 4.39 -1.23) (layer F.Fab) (width 0.1))
-    (fp_line (start -2.58 -2.62) (end 7.66 -2.62) (layer F.SilkS) (width 0.12))
-    (fp_line (start -2.58 2.021) (end 7.66 2.021) (layer F.SilkS) (width 0.12))
-    (fp_line (start -2.58 -2.62) (end -2.58 2.021) (layer F.SilkS) (width 0.12))
-    (fp_line (start 7.66 -2.62) (end 7.66 2.021) (layer F.SilkS) (width 0.12))
-    (fp_line (start -2.58 -1.11) (end 7.66 -1.11) (layer F.SilkS) (width 0.12))
-    (fp_line (start 0.69 -2.62) (end 0.69 -1.11) (layer F.SilkS) (width 0.12))
-    (fp_line (start 4.391 -2.62) (end 4.391 -1.11) (layer F.SilkS) (width 0.12))
-    (fp_line (start -2.71 -2.75) (end -2.71 2.16) (layer F.CrtYd) (width 0.05))
-    (fp_line (start -2.71 2.16) (end 7.79 2.16) (layer F.CrtYd) (width 0.05))
-    (fp_line (start 7.79 2.16) (end 7.79 -2.75) (layer F.CrtYd) (width 0.05))
-    (fp_line (start 7.79 -2.75) (end -2.71 -2.75) (layer F.CrtYd) (width 0.05))
-    (pad 1 thru_hole rect (at 0 0 270) (size 1.8 1.8) (drill 1) (layers *.Cu *.Mask)
-      (net 37 "Net-(Q4-Pad1)"))
-    (pad 2 thru_hole oval (at 2.54 0 270) (size 1.8 1.8) (drill 1) (layers *.Cu *.Mask)
-      (net 32 /LED1_R))
-    (pad 3 thru_hole oval (at 5.08 0 270) (size 1.8 1.8) (drill 1) (layers *.Cu *.Mask)
-      (net 5 GND))
-    (model ${KISYS3DMOD}/Package_TO_SOT_THT.3dshapes/TO-220-3_Vertical.step
-      (at (xyz 0 0 0))
-      (scale (xyz 1.1 1 1))
-      (rotate (xyz 0 0 0))
-    )
-  )
-  (module Modules:Arduino_Nano (layer F.Cu)
+  (module Module:Arduino_Nano (layer F.Cu)
     (at 158.74 92 180)
     (descr "Arduino Nano, http://www.mouser.com/pdfdocs/Gravitech_Arduino_Nano3_0.pdf")
@@
     (pad 16 thru_hole oval (at 15.24 35.56 180) (size 1.6 1.6) (drill 0.8) (layers *.Cu *.Mask)
       (net 27 /ar_LED_BuiltIn))
+    (model ${GOINK13}/3D/Arduino_nanoRev3.STEP
+      (offset (xyz 0 0 2.54))
+      (scale (xyz 1 1 1))
+      (rotate (xyz -90 0 90))
+    )
+  )
+  (module TO_SOT_Packages_THT:TO-220-3_Vertical (layer F.Cu)
+    (at 161 101 270)
+    (descr "TO-220-3, Vertical, RM 2.54mm")
+    (tags "TO-220-3 Vertical RM 2.54mm")
+    (fp_text reference Q4 (at 2.54 -3.62 270) (layer F.SilkS)
+      (effects (font (size 1 1) (thickness 0.15)))
+    )
+    (fp_text value IRFZ44N (at 2.54 3.92 270) (layer F.Fab) hide
+      (effects (font (size 1 1) (thickness 0.15)))
+    )
+    (fp_text user %R (at 2.54 -3.62 270) (layer F.Fab) hide
+      (effects (font (size 1 1) (thickness 0.15)))
+    )
+    (fp_line (start -2.46 -2.5) (end -2.46 1.9) (layer F.Fab) (width 0.1))
+    (fp_line (start -2.46 1.9) (end 7.54 1.9) (layer F.Fab) (width 0.1))
+    (fp_line (start 7.54 1.9) (end 7.54 -2.5) (layer F.Fab) (width 0.1))
+    (fp_line (start 7.54 -2.5) (end -2.46 -2.5) (layer F.Fab) (width 0.1))
+    (fp_line (start -2.46 -1.23) (end 7.54 -1.23) (layer F.Fab) (width 0.1))
+    (fp_line (start 0.69 -2.5) (end 0.69 -1.23) (layer F.Fab) (width 0.1))
+    (fp_line (start 4.39 -2.5) (end 4.39 -1.23) (layer F.Fab) (width 0.1))
+    (fp_line (start -2.58 -2.62) (end 7.66 -2.62) (layer F.SilkS) (width 0.12))
+    (fp_line (start -2.58 2.021) (end 7.66 2.021) (layer F.SilkS) (width 0.12))
+    (fp_line (start -2.58 -2.62) (end -2.58 2.021) (layer F.SilkS) (width 0.12))
+    (fp_line (start 7.66 -2.62) (end 7.66 2.021) (layer F.SilkS) (width 0.12))
+    (fp_line (start -2.58 -1.11) (end 7.66 -1.11) (layer F.SilkS) (width 0.12))
+    (fp_line (start 0.69 -2.62) (end 0.69 -1.11) (layer F.SilkS) (width 0.12))
+    (fp_line (start 4.391 -2.62) (end 4.391 -1.11) (layer F.SilkS) (width 0.12))
+    (fp_line (start -2.71 -2.75) (end -2.71 2.16) (layer F.CrtYd) (width 0.05))
+    (fp_line (start -2.71 2.16) (end 7.79 2.16) (layer F.CrtYd) (width 0.05))
+    (fp_line (start 7.79 2.16) (end 7.79 -2.75) (layer F.CrtYd) (width 0.05))
+    (fp_line (start 7.79 -2.75) (end -2.71 -2.75) (layer F.CrtYd) (width 0.05))
+    (pad 1 thru_hole rect (at 0 0 270) (size 1.8 1.8) (drill 1) (layers *.Cu *.Mask)
+      (net 37 "Net-(Q4-Pad1)"))
+    (pad 2 thru_hole oval (at 2.54 0 270) (size 1.8 1.8) (drill 1) (layers *.Cu *.Mask)
+      (net 32 /LED1_R))
+    (pad 3 thru_hole oval (at 5.08 0 270) (size 1.8 1.8) (drill 1) (layers *.Cu *.Mask)
+      (net 5 GND))
+    (model ${KISYS3DMOD}/Package_TO_SOT_THT.3dshapes/TO-220-3_Vertical.step
+      (at (xyz 0 0 0))
+      (scale (xyz 1.1 1 1))
+      (rotate (xyz 0 0 0))
+    )
   )
   (module Capacitors_ThroughHole:CP_Radial_D8.0mm_P3.50mm (layer F.Cu)
